File: hstat.kicad_pcb (KiCad board)
At the start: 2 copper layers, 116.3 x 73 mm, 78 parts, among them J1 BAT, J3 TMP2, J4 OUT-1, J5 OUT-2, J6 USB_C_Receptacle_USB2.0_16P, K1 EE2-3TNUH, Q1 AO3401A, Q2 BC817-40, Q3 BC817-40, Q4 BC817-40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

Commit message: Add logos etc.
Parts:
- added G***: LOGO, logo:cedar-creek-electronics, B.Cu at (109.6, 81.4)
Other:
- board text added: "JLCJLCJLCJLC"
- board text added: "hstat - v1.0"

Commit message: new schematic
Parts:
- removed C14: 100nF/16V, Capacitor_SMD:C_0805_2012Metric
- removed U5: BME280, Package_LGA:Bosch_LGA-8_2.5x2.5mm_P0.65mm_ClockwisePinNumbering
- added R22: 4.7k, Resistor_SMD:R_0805_2012Metric, F.Cu at (129.2, 55.2)
- added R23: 4.7k, Resistor_SMD:R_0805_2012Metric, F.Cu at (129.2, 59.0)
- added U8: HDC1080, Package_SON:Texas_PWSON-N6, F.Cu at (142.6, 114.0)
- U1: footprint Package_TO_SOT_SMD:TSOT-23-6 -> Package_TO_SOT_SMD:SOT-23-6
- moved C13 7.41 mm to (146.2, 113.9), turned to 90 degrees
Connections:
- J6 pad A5: (no net) -> unconnected-(J6-CC1-PadA5)
- J6 pad A8: (no net) -> unconnected-(J6-SBU1-PadA8)
- J6 pad B5: (no net) -> unconnected-(J6-CC2-PadB5)
- J6 pad B8: (no net) -> unconnected-(J6-SBU2-PadB8)
Routing:
- net /TEMP1-CS: track 93.9 -> 0.00 mm, vias 2 -> 0
- net /SPI-SCK: track 105.1 -> 22.8 mm, vias 3 -> 1
- net /SPI-MISO: track 106.0 -> 24.4 mm, vias 3 -> 1
- net /SPI-MOSI: track 102.4 -> 21.0 mm, vias 3 -> 1
- net /I2C-SCL: track 58.0 -> 123.0 mm, vias 1 -> 2
- net /I2C-SDA: track 57.1 -> 118.9 mm, vias 1 -> 2
- net +3V3: track 398.1 -> 386.5 mm, vias 9 -> 8
- net GND: track 21.6 -> 27.4 mm
- net /TEMP2-DATA: track 31.9 -> 34.5 mm
- net /BTN1: track 61.7 -> 63.1 mm
- net /TS-INT: track 54.8 -> 56.1 mm
- net /GPIO2: track 106.1 -> 106.9 mm
Other:
- outline, holes or cut-outs redrawn
