File: V2/hstat-v2.kicad_sch (KiCad schematic)
At the start: 181 parts, among them J1 USB_C_Receptacle_USB2.0_16P, J2 Conn_01x03, J3 Conn_01x03, J4 Conn_01x03, K1 EE2-3TNUH, Q1 BC817, Q10 SIS412DN, Q11 Si7617DN, Q12 BC817, Q13 BC817, Q2 BC817, Q4 Q_NMOS, Q5 Q_NMOS, Q6 Si1308EDL, Q7 Si7617DN, Q8 Si7617DN, Q9 SIS412DN, SW1 SW_Push, SW3 SW_Push, SW4 SW_Push, SW5 SW_Push, U1 CH340T, U10 EL817, U11 EL817, U12 TPS61165DBV, U13 DS18B20Z, U2 ESP32-WROVER-E, U3 SHT4x, U4 BQ7791506PWR, U5 BQ24610, U6 AP63203WU, U7 DS18B20Z, U8 LTR-303ALS-01, Y1 12MHz

Commit message: Before board split
Parts:
- removed BT2, BT3, BT4: 18650, MH_connectors:254-keystone-18650, symbol *partsbox:254
- removed C14, C15, C19, C20, C21, C22, C33, C35, C36, C39, C42, C43, C44, C45: 100nF, symbol Device:C_Small
- removed C17: 1uF, symbol Device:C_Small
- removed C34: 2.2uF, Capacitor_SMD:C_1206_3216Metric_Pad1.33x1.80mm_HandSolder, symbol Device:C_Polarized_Small_US
- removed C37, C40, C41: 1uF, Capacitor_SMD:C_1206_3216Metric_Pad1.33x1.80mm_HandSolder, symbol Device:C_Polarized_Small_US
- removed C38: 0.056uF, Capacitor_SMD:C_1206_3216Metric_Pad1.33x1.80mm_HandSolder, symbol Device:C_Polarized_Small_US
- removed C46, C47, C48, C50: 10uF, Capacitor_SMD:C_1206_3216Metric_Pad1.33x1.80mm_HandSolder, symbol Device:C_Polarized_Small_US
- removed C49: 22pF, symbol Device:C_Small
- removed C51: 10uF, Capacitor_SMD:C_0805_2012Metric, symbol Device:C_Small
- removed C52: 100nF/16V, Capacitor_SMD:C_0805_2012Metric, symbol Device:C_Small
- removed C53, C54: 22uF/LOW ESR, Capacitor_SMD:C_1206_3216Metric_Pad1.33x1.80mm_HandSolder, symbol Device:C_Polarized_Small_US
- removed D10: LED, symbol Device:LED
- removed D13: BAT54, symbol Device:D_Schottky
- removed F1: 2A, symbol Device:Fuse
- removed L3: 6.8uH, symbol Device:L
- removed L4: 2.2uH, Inductor_SMD:L_Taiyo-Yuden_NR-60xx_HandSoldering, symbol Device:L_Iron_Small
- removed Q10, Q9: SIS412DN, symbol MH_transistors:SIS412DN
- removed Q11, Q7, Q8: Si7617DN, Package_SO:Vishay_PowerPAK_1212-8_Single, symbol Transistor_FET:Si7617DN
- removed Q4, Q5: Q_NMOS, symbol Device:Q_NMOS
- removed R11, R12, R13, R14, R15, R16: 1K, symbol Device:R_US
- removed R17: 1m, symbol Device:R_US
- removed R18, R19: 1M, symbol Device:R_US
- removed R20: 4.5k, symbol Device:R_US
- removed R21, R44: 1k, symbol Device:R_US
- removed R22, R23, R41: 100R, symbol Device:R_US
- removed R24, R25, R39: 10k, symbol Device:R_US
- removed R26, R31, R36, R37, R46: 100k, symbol Device:R_US
- removed R27: 450k, symbol Device:R_US
- removed R32: 2R, symbol Device:R_US
- removed R33, R45: 10m, Resistor_SMD:R_0603_1608Metric, symbol *partsbox:0603-0ohm
- removed R38: 32.4k, symbol Device:R_US
- removed R40: 22.1k, symbol Device:R_US
- removed R42: 9.31k, symbol Device:R_US
- removed R43: 430k, symbol Device:R_US
- removed R47, R48: 500k, Resistor_SMD:R_0603_1608Metric, symbol *partsbox:0603-0ohm
- removed TH1: 103AT, symbol Device:Thermistor_NTC_US
- removed U4: BQ7791506PWR, Package_SO:TSSOP-24_4.4x7.8mm_P0.65mm, symbol *partsbox:BQ7791506PWR
- removed U5: BQ24610, Package_DFN_QFN:VQFN-24-1EP_4x4mm_P0.5mm_EP2.45x2.45mm, symbol Battery_Management:BQ24610
- removed U6: AP63203WU, Package_TO_SOT_SMD:TSOT-23-6, symbol Regulator_Switching:AP63203WU
- added BT5, BT6, BT7, BT8: 18650, MH_connectors:254-keystone-18650, symbol *partsbox:254
- added C11: 4.7uF, Capacitor_SMD:C_0805_2012Metric, symbol Device:C_Small
- added C14: 12pF, symbol Device:C_Trim
- added C15: 100nF, Capacitor_SMD:C_0603_1608Metric, symbol *partsbox:0603-1uF
- added C17: 1uF, Capacitor_SMD:C_0603_1608Metric, symbol *partsbox:0603-1uF
- added D10, D3: D, symbol Device:D
- added JP2: SolderJumper_3_Bridged12, symbol Jumper:SolderJumper_3_Bridged12
- added JP3: 1.5A, symbol Jumper:SolderJumper_2_Open
- added JP4: 0.5A, symbol Jumper:SolderJumper_2_Open
- added JP5: 1A, symbol Jumper:SolderJumper_2_Bridged
- added JP6: EN2, symbol Jumper:SolderJumper_3_Bridged12
- added JP7: EN1, symbol Jumper:SolderJumper_3_Bridged12
- added R11, R39: 0R, Resistor_SMD:R_0603_1608Metric, symbol *partsbox:0603-10Kohm
- added R31: 500R, Resistor_SMD:R_0603_1608Metric, symbol *partsbox:0603-10Kohm
- added R32, R36: 1k, Resistor_SMD:R_0603_1608Metric, symbol *partsbox:0603-10Kohm
- added R33: 2k, Resistor_SMD:R_0603_1608Metric, symbol *partsbox:0603-10Kohm
- added R37, R38: 10k, Resistor_SMD:R_0603_1608Metric, symbol *partsbox:0603-10Kohm
- added SW2: SW_DPST, symbol Switch:SW_DPST
- added TP1: CLK_OUT, symbol Connector:TestPoint
- added TP2: CHG_CURR, symbol Connector:TestPoint
- added U4: AP7361C-33E, Package_TO_SOT_SMD:SOT-223-3_TabPin2, symbol Regulator_Linear:AP7361C-33E
- added U5: BQ24074RGT, Package_DFN_QFN:VQFN-16-1EP_3x3mm_P0.5mm_EP1.6x1.6mm, symbol Battery_Management:BQ24074RGT
- added U6: PCF8563T, Package_SO:SOIC-8_3.9x4.9mm_P1.27mm, symbol Timer_RTC:PCF8563T
- added U9: MAX17048G_T10, MAX17048G_T10:SON50P200X200X80-9N, symbol MH_ics:MAX17048G_T10
- added Y2: 32.768khz, symbol Device:Crystal_GND24_Small
- BT1: value 18650 -> CR
- C13: value 100nF -> 4.7uF; footprint (none) -> Capacitor_SMD:C_0805_2012Metric; JLCPCB PN (none) -> C15850
- C16: value 100nF -> 4.7uF/25V
- C18: value 1uF -> 4.7uF/25V
- D11: value LED -> RED
- D9: value LED -> GREEN
- R34: value 1k -> 1.5k
- R35: value 100k -> 1.5k
Connections:
- net +3V3: now also C13.1, D3.2 (A), JP2.3 (B), U4.3 (VO)
- net +BATT: now also C16.1, BT5.1 (+), BT6.1 (+), BT7.1 (+), BT8.1 (+), C15.2, U5.2 (BAT), U5.3 (BAT), U9.2 (CELL), U9.3 (VDD); no longer BT1.1 (+)
- net GND: now also BT1.2 (-), C16.2, C18.2, TH2.1, BT5.2 (-), BT6.2 (-), BT7.2 (-), BT8.2 (-), C11.2, C14.2, C15.1, C17.2, JP3.1 (A), JP4.1 (A), JP5.1 (A), JP6.1 (A), JP7.3 (B), R36.2, R37.2, R38.2, R39.2, U4.2 (GND), U5.17 (VSS), U5.8 (VSS), U6.4 (VSS), U9.1 (CTG), U9.4 (GND), U9.6 (QSTRT), U9.9 (EP), Y2.2 (G), Y2.4 (G); no longer C18.1, TH2.2
- net VBUS: now also SW2.4; no longer D11.2 (A), D9.2 (A), J1.A4 (VBUS), J1.A9 (VBUS), J1.B4 (VBUS), J1.B9 (VBUS)
- net at R34.1: now also D9.2 (A)
- net VPP: now reaches R34.2
- net VPP: now also R35.2, C11.1, JP2.1 (A), JP6.3 (B), JP7.1 (A), SW2.2, U4.1 (VI)
- net at D9.1 (K): now also U5.7 (~{PGOOD})
- net at D11.1 (K): now also U5.9 (~{CHG})
- net VDC: no longer names the net of C12.1, L5.1, U12.1 (VIN)
- net VDC: now also JP2.2 (C)
- net VREF: no longer names the net of R35.1
- net VREF: now also D11.2 (A)
- new net: C14.1, U6.1 (OSCI), Y2.1
- new net: R31.1, R32.1, R33.1, TP2.1, U5.16 (ISET)
- new net: JP3.2 (B), R31.2
- new net: JP4.2 (B), R33.2
- new net: U6.2 (OSCO), Y2.3
- new net: TP1.1, U6.7 (CLKO)
- new net: D3.1 (K), R11.1, U6.8 (VDD)
- new net: JP5.2 (B), R32.2
- new net: R37.1, U5.4 (~{CE})
- new net: D10.1 (K), R11.2
- new net: TH2.2, U5.1 (TS)
- new net: BT1.1 (+), D10.2 (A)
- new net: R38.1, U5.15 (ITERM)
- new net: JP7.2 (C), U5.6 (EN1)
- new net: R36.1, U5.12 (ILIM)
- new net: JP6.2 (C), U5.5 (EN2)
- new net: R39.1, U5.14 (TMR)
- new net VBUS_SW: C17.1, J1.A4 (VBUS), J1.A9 (VBUS), J1.B4 (VBUS), J1.B9 (VBUS), SW2.3, U5.13 (IN)
- new net VPP_SW: C18.1, SW2.1, U5.10 (OUT), U5.11 (OUT)
- no-connect marks 10 -> 7
Other:
- note added: "Fuel Gauge"
- note removed: "Battery Protection"
- moved on the sheet: C10, H1, H2, H3, H4, R51, R52, R53, R54, SW3, SW4, SW5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

Commit message: Main board in progress
Other:
- note added: "RTC"
Changed lines of the file:
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@@
+		)
+	)
+	(text "RTC"
+		(exclude_from_sim no)
+		(at 330.2 93.218 0)
+		(effects
+			(font
+				(size 3.81 3.81)
+				(thickness 1.016)
+				(bold yes)
+				(color 0 194 0 1)
+			)
 		)
 	)
