File: V2/main_board/main_board.kicad_sch (KiCad schematic)
At the start: 86 parts, among them J1 USB_C_Receptacle_USB2.0_16P, J2 Conn_01x03, J3 Conn_01x03, J4 Conn_01x03, J5 Conn_01x12, J6 Conn_01x12, K1 EE2-3TNUH, Q12 BC817, Q13 BC817, SW2 SW_Push, SW3 SW_Slide_DPDT, SW4 SW_Push, U10 EL817, U11 EL817, U13 DS18B20Z, U3 SHT4x, U4 AP7361C-33E, U5 BQ24074RGT, U6 PCF8563T, U7 ESP32-S3-WROOM-2, U8 DS18B20Z, U9 MAX17048G_T10, Y1 32.768kHz

Commit message: Initial component placement done.
Parts:
- removed BT5, BT6, BT7, BT8: 18650, MH_connectors:254-keystone-18650, symbol *partsbox:254
- removed C11, C13: 4.7uF, Capacitor_SMD:C_0805_2012Metric, symbol Device:C_Small
- removed C14: 12pF, symbol Device:C_Trim
- removed C15: 100nF, Capacitor_SMD:C_0603_1608Metric, symbol *partsbox:0603-1uF
- removed C16, C18: 4.7uF/25V, symbol Device:C_Small
- removed C17: 1uF, Capacitor_SMD:C_0603_1608Metric, symbol *partsbox:0603-1uF
- removed C55: 100uF, Capacitor_SMD:C_1206_3216Metric_Pad1.33x1.80mm_HandSolder, symbol Device:C_Polarized_Small_US
- removed C56: 100uF, Capacitor_SMD:CP_Elec_8x10, symbol Device:C_Polarized_Small_US
- removed D10, D3: M7, symbol Device:D
- removed D11: RED, symbol Device:LED
- removed D12: D, symbol Device:D
- removed D14: D, Diode_SMD:D_SMA, symbol Device:D
- removed D9: GREEN, symbol Device:LED
- removed F2: 2A, symbol Device:Fuse
- removed F3: 2A, Fuse:Fuse_Schurter_UMZ250, symbol Device:Fuse
- removed J2, J3, J4: Conn_01x03, symbol Connector_Generic:Conn_01x03
- removed K1: EE2-3TNUH, Relay_SMD:Relay_DPDT_Kemet_EE2_NUH_DoubleCoil, symbol Relay:EE2-3TNUH
- removed Q12, Q13: BC817, Package_TO_SOT_SMD:SOT-23, symbol Transistor_BJT:BC817
- removed R11, R39: 0R, Resistor_SMD:R_0603_1608Metric, symbol *partsbox:0603-10Kohm
- removed R3: 10K, Resistor_SMD:R_0603_1608Metric, symbol *partsbox:0603-10Kohm
- removed R31: 500R, Resistor_SMD:R_0603_1608Metric, symbol *partsbox:0603-10Kohm
- removed R32, R36: 1k, Resistor_SMD:R_0603_1608Metric, symbol *partsbox:0603-10Kohm
- removed R33: 2k, Resistor_SMD:R_0603_1608Metric, symbol *partsbox:0603-10Kohm
- removed R34, R35: 1.5k, symbol Device:R_US
- removed R37, R38: 10k, Resistor_SMD:R_0603_1608Metric, symbol *partsbox:0603-10Kohm
- removed R4: 0R, Resistor_SMD:R_0603_1608Metric, symbol *partsbox:0603-0ohm
- removed R49, R50: 120R, symbol Device:R_US
- removed R5: 1K, Resistor_SMD:R_0603_1608Metric, symbol *partsbox:0603-1Kohm
- removed R6: 510R, Resistor_SMD:R_0603_1608Metric, symbol *partsbox:0603-510ohm
- removed SW3: SW_Slide_DPDT, Button_Switch_THT:SW_E-Switch_EG2219_DPDT_Angled, symbol Switch:SW_Slide_DPDT
- removed TH2: 103AT, symbol Device:Thermistor_NTC_US
- removed U10: EL817, Package_DIP:SMDIP-4_W7.62mm, symbol Isolator:EL817
- removed U11: EL817, Package_DIP:DIP-4_W7.62mm, symbol Isolator:EL817
- removed U3: SHT4x, Sensor_Humidity:Sensirion_DFN-4_1.5x1.5mm_P0.8mm_SHT4x_NoCentralPad, symbol *partsbox:SHT41-AD1B-R2
- removed U4: AP7361C-33E, Package_TO_SOT_SMD:SOT-223-3_TabPin2, symbol Regulator_Linear:AP7361C-33E
- removed U6: PCF8563T, Package_SO:SOIC-8_3.9x4.9mm_P1.27mm, symbol Timer_RTC:PCF8563T
- removed U7: ESP32-S3-WROOM-2, RF_Module:ESP32-S3-WROOM-2, symbol RF_Module:ESP32-S3-WROOM-2
- removed U9: MAX17048G_T10, MAX17048G_T10:SON50P200X200X80-9N, symbol MH_ics:MAX17048G_T10
- removed Y1: 32.768kHz, Crystal:Crystal_SMD_3215-2Pin_3.2x1.5mm, symbol Device:Crystal_Small
- added BT1, BT2, BT3, BT4: 18650, MH_connectors:1043-keystone-18650, symbol *partsbox:1043
- added C1: 1uF, Capacitor_SMD:C_0603_1608Metric, symbol *partsbox:0603-1uF
- added C2, C3, C4, C5: 4.7uF, Capacitor_SMD:C_0603_1608Metric, symbol *partsbox:0603-4.7uF-25V
- added C6: 100nF, Capacitor_SMD:C_0603_1608Metric, symbol *partsbox:0603-100nF
- added C7, C8: 100uF, Capacitor_SMD:CP_Elec_8x10, symbol *partsbox:UUD1H101MNL1GS
- added C9: 4.5/20pF, Capacitor_SMD:C_Trimmer_Voltronics_JZ, symbol *partsbox:JZ200HV
- added D2: RED, LED_SMD:LED_0805_2012Metric, symbol *partsbox:NCD0805R1
- added D3, D4, D5, D6: M7, Diode_SMD:D_SMA, symbol *partsbox:M7
- added F1, F2: 2A, Fuse:Fuse_Schurter_UMZ250, symbol *partsbox:3404.2419.11
- added J3: OUT_1, TerminalBlock_Phoenix:TerminalBlock_Phoenix_MKDS-1,5-3_1x03_P5.00mm_Horizontal, symbol *partsbox:691137710003
- added J4: OUT_2, TerminalBlock_Phoenix:TerminalBlock_Phoenix_MKDS-1,5-3_1x03_P5.00mm_Horizontal, symbol *partsbox:691137710003
- added J5: EXT_TEMP, MH_connectors:PHOENIX_1771033, symbol *partsbox:1771033
- added K1: EE2-3TNUH, Relay_SMD:Relay_DPDT_Kemet_EE2_NUH_DoubleCoil, symbol *partsbox:EE2-3TNUH
- added Q1, Q2: BC817, Package_TO_SOT_SMD:SOT-23, symbol *partsbox:BC817-40
- added R1, R2: 10K, Resistor_SMD:R_0603_1608Metric, symbol *partsbox:0603-10Kohm
- added R10, R11: 120R, Resistor_SMD:R_0603_1608Metric, symbol *partsbox:0603-120ohm
- added R12, R3: 0R, Resistor_SMD:R_0603_1608Metric, symbol *partsbox:0603-0ohm
- added R4, R6: 1K, Resistor_SMD:R_0603_1608Metric, symbol *partsbox:0603-1Kohm
- added R5: 510R, Resistor_SMD:R_0603_1608Metric, symbol *partsbox:0603-510ohm
- added R9: 1.5K, Resistor_SMD:R_0603_1608Metric, symbol *partsbox:0603-1.5Kohm
- added SW1: SW_Slide_DPDT, Button_Switch_THT:SW_E-Switch_EG2219_DPDT_Angled, symbol *partsbox:EG2219
- added TP4: TXD, TestPoint:TestPoint_Pad_2.0x2.0mm, symbol Connector:TestPoint
- added TP5: RXD, TestPoint:TestPoint_Pad_2.0x2.0mm, symbol Connector:TestPoint
- added TP6: IO45, TestPoint:TestPoint_Pad_2.0x2.0mm, symbol Connector:TestPoint
- added TP7: IO46, TestPoint:TestPoint_Pad_2.0x2.0mm, symbol Connector:TestPoint
- added TP8: IO3, TestPoint:TestPoint_Pad_2.0x2.0mm, symbol Connector:TestPoint
- added U10: ESP32-S3-WROOM-2, RF_Module:ESP32-S3-WROOM-2, symbol *partsbox:ESP32-S3-WROOM-2-N32R16V
- added U2: AP7361C-33E, Package_TO_SOT_SMD:SOT-223-3_TabPin2, symbol *partsbox:AP7361C-33E-13
- added U3: MAX17048G_T10, MH_ics:SON50P200X200X80-9N, symbol *partsbox:MAX17048G+T10
- added U4, U5: EL817, Package_DIP:SMDIP-4_W7.62mm, symbol *partsbox:EL8171S1(TU)-G
- added U6: PCF8563T, Package_SO:SOIC-8_3.9x4.9mm_P1.27mm, symbol *partsbox:PCF8563T/5,518
- added Y1: 32.768khz, Crystal:Crystal_SMD_3215-2Pin_3.2x1.5mm, symbol *partsbox:Q13FC13500004
- H1, H2, H3, H4: footprint (none) -> MountingHole:MountingHole_3.2mm_M3_ISO7380_Pad_TopBottom
- JP1: renamed from JP7; footprint (none) -> Jumper:SolderJumper-3_P1.3mm_Bridged12_RoundedPad1.0x1.5mm
- JP2: renamed from JP6; footprint (none) -> Jumper:SolderJumper-3_P1.3mm_Bridged12_RoundedPad1.0x1.5mm
- JP3: footprint (none) -> Jumper:SolderJumper-2_P1.3mm_Open_RoundedPad1.0x1.5mm
- JP4: renamed from JP5; footprint (none) -> Jumper:SolderJumper-2_P1.3mm_Bridged_RoundedPad1.0x1.5mm
- JP5: renamed from JP4; footprint (none) -> Jumper:SolderJumper-2_P1.3mm_Open_RoundedPad1.0x1.5mm
- TP1: renamed from TP2; footprint (none) -> TestPoint:TestPoint_Pad_2.0x2.0mm
- TP2: renamed from TP3; footprint (none) -> TestPoint:TestPoint_Pad_2.0x2.0mm
- TP3: renamed from TP1; footprint (none) -> TestPoint:TestPoint_Loop_D2.54mm_Drill1.5mm_Beaded
- renumbered BT1 to BT5, C20 to C10, C12 to C11, C9 to C12, C10 to C13, J5 to J1, J6 to J2, J1 to J6, R12 to R13, R13 to R14, R1 to R15, R2 to R16, SW4 to SW3, U5 to U1, U13 to U8, U8 to U9
Connections:
- net TS_SCL is gone; now on net ONEWIRE: J2.7 (Pin_7)
- net TS_SDA is gone; now on net TS_INT: J2.8 (Pin_8)
- net +3V3: now also C5.1, C7.1, C8.1, D3.1 (K), D4.1 (K), D5.2 (A), J5.1 (Pin_1), K1.1, K1.6, U10.2 (3V3), U2.3 (VO), U4.4, U5.4
- net +BATT: now also BT1.1 (+), BT2.1 (+), BT3.1 (+), BT4.1 (+), C3.1, C6.1, U3.2 (CELL), U3.3 (VDD)
- net ADDR_LED: now also J1.10 (Pin_10), U10.4 (IO4); no longer J1.11 (Pin_11)
- net ALS_INT: now also U10.11 (IO18); no longer J1.7 (Pin_7)
- net BOOT0: now also U10.27 (IO0)
- net BTN1: now also U10.34 (MTDI/IO41)
- net BTN2: now also U10.35 (MTMS/IO42)
- net BTN3: now also U10.24 (IO47)
- net BTN4: now also U10.25 (IO48)
- net D+: now also U10.14 (USB_D+/IO20)
- net D-: now also U10.13 (USB_D-/IO19)
- net DISP_BUSY: now also U10.7 (IO7)
- net DISP_CS: now also U10.18 (IO10)
- net DISP_D/C: now also U10.17 (IO9)
- net DISP_RES: now also U10.12 (IO8)
- net DISP_SCLK: now also U10.20 (IO12)
- net DISP_SDA: now also U10.19 (IO11)
- net GND: now also TH1.2, BT1.2 (-), BT2.2 (-), BT3.2 (-), BT4.2 (-), C1.2, C2.1, C3.2, C4.2, C5.2, C6.2, C9.2, J5.3 (Pin_3), Q1.2 (E), Q2.2 (E), R1.2, R2.2, R3.2, R4.2, U10.1 (GND), U10.40 (GND), U10.41 (GND), U2.2 (GND), U3.1 (CTG), U3.4 (GND), U3.6 (QSTRT), U3.9 (EP), U4.2, U5.2, U6.4 (VSS)
- net I2C_SCL: now also U10.38 (IO2), U3.7 (SCL), U6.6 (SCL)
- net I2C_SDA: now also U10.39 (IO1), U3.8 (SDA), U6.5 (SDA)
- net LED_G: now also J1.9 (Pin_9), U10.32 (MTCK/IO39); no longer J1.10 (Pin_10)
- net ONEWIRE: now also J5.2 (Pin_2), U10.31 (IO38); no longer J2.11 (Pin_11)
- net RELAY_RESET: now also R11.1, U10.6 (IO6)
- net RELAY_SET: now also R10.1, U10.5 (IO5)
- net RESET: now also U10.3 (EN)
- net RTC_INT: now also U10.23 (IO21), U6.3 (~{INT})
- net SCL: now also J1.8 (Pin_8), U10.22 (IO14); no longer J1.9 (Pin_9)
- net SDA: now also J1.7 (Pin_7), U10.8 (IO15); no longer J1.8 (Pin_8)
- net SPI_MISO: now also U10.21 (IO13)
- net TS_INT: now also U10.9 (IO16); no longer J2.9 (Pin_9)
- net TS_RST: now also J2.9 (Pin_9), U10.10 (IO17); no longer J2.10 (Pin_10)
- net VBUS: now also C1.1, SW1.5 (B)
- net VBUS_SW: now also SW1.4 (A)
- net VPP: now also R8.1, C4.1, R9.2, SW1.2 (B), U2.1 (VI)
- net VPP_SW: now also C2.2, SW1.3 (C)
- net at TP2.1: now also U3.5 (~{ALERT})
- net at TP1.1, U1.16 (ISET): now also R7.1, R5.1, R6.1
- net at JP3.2 (B): now also R5.2
- net at JP5.2 (B): now also R7.2
- net at TH1.1: now also U1.1 (TS)
- net at R8.2: now also D1.1 (K)
- net at TP3.1: now also U6.7 (CLKO)
- net at JP4.2 (B): now also R6.2
- net at U1.4 (~{CE}): now also R2.1
- net at U1.7 (~{PGOOD}): now also D1.2 (A)
- net at U1.9 (~{CHG}): now also D2.2 (A)
- net at BT5.1 (+): now also D6.2 (A)
- net at U1.15 (ITERM): now also R1.1
- net at U1.12 (ILIM): now also R4.1
- net at U1.14 (TMR): now also R3.1
- new net: TP8.1, U10.15 (IO3)
- new net: R10.2, U4.1
- new net: Q1.1 (B), U4.3
- new net: F2.1, K1.9
- new net: F2.2, J3.2 (Pin_2)
- new net: J3.1 (Pin_1), K1.3
- new net: J3.3 (Pin_3), K1.5
- new net: F1.1, K1.4
- new net: F1.2, J4.2 (Pin_2)
- new net: R11.2, U5.1
- new net: D5.1 (K), R12.1, U6.8 (VDD)
- new net: D6.1 (K), R12.2
- new net: C7.2, D3.2 (A), K1.7, Q2.3 (C)
- new net: Q2.1 (B), U5.3
- new net: C8.2, D4.2 (A), K1.12, Q1.3 (C)
- new net: U6.2 (OSCO), Y1.1
- new net: C9.1, U6.1 (OSCI), Y1.2
- new net: J4.1 (Pin_1), K1.10
- new net: J4.3 (Pin_3), K1.8
- new net: D2.1 (K), R9.1
- new net: TP7.1, U10.16 (IO46)
- new net: TP6.1, U10.26 (IO45)
- new net LED_PWM: J1.11 (Pin_11), U10.33 (MTDO/IO40)
- new net PRESENCE_RX: J2.11 (Pin_11), TP4.1, U10.37 (TXD0/IO43)
- new net PRESENCE_TX: J2.10 (Pin_10), TP5.1, U10.36 (RXD0/IO44)
Other:
- moved on the sheet: U8, U9

Commit message: In progress
Parts:
- removed BT5: RTC_BAT, Battery:BatteryHolder_Keystone_1057_1x2032, symbol *partsbox:254
- removed C7, C8: 100uF, Capacitor_SMD:CP_Elec_8x10, symbol *partsbox:UUD1H101MNL1GS
- removed D1: GREEN, LED_SMD:LED_0805_2012Metric, symbol *partsbox:KT-0805G
- removed D2: RED, LED_SMD:LED_0805_2012Metric, symbol *partsbox:NCD0805R1
- removed F1, F2: 2A, Fuse:Fuse_Schurter_UMZ250, symbol *partsbox:3404.2419.11
- removed J1, J2: Conn_01x12, Connector_PinHeader_2.54mm:PinHeader_1x12_P2.54mm_Vertical_SMD_Pin1Left, symbol *partsbox:TSM-112-01-SM-SV
- removed J3: OUT_1, TerminalBlock_Phoenix:TerminalBlock_Phoenix_MKDS-1,5-3_1x03_P5.00mm_Horizontal, symbol *partsbox:691137710003
- removed J4: OUT_2, TerminalBlock_Phoenix:TerminalBlock_Phoenix_MKDS-1,5-3_1x03_P5.00mm_Horizontal, symbol *partsbox:691137710003
- removed K1: EE2-3TNUH, Relay_SMD:Relay_DPDT_Kemet_EE2_NUH_DoubleCoil, symbol *partsbox:EE2-3TNUH
- removed R8, R9: 1.5K, Resistor_SMD:R_0603_1608Metric, symbol *partsbox:0603-1.5Kohm
- removed TP6: IO45, TestPoint:TestPoint_Pad_2.0x2.0mm, symbol Connector:TestPoint
- removed TP7: IO46, TestPoint:TestPoint_Pad_2.0x2.0mm, symbol Connector:TestPoint
- added BT5: CR2032, Battery:BatteryHolder_Keystone_1058_1x2032, symbol *partsbox:1058
- added D1, D2: M7, Diode_SMD:D_SMA, symbol *partsbox:M7
- added F1, F2: 10A, Fuse:Fuse_Schurter_UMT250, symbol *partsbox:3403.0176.11
- added J1, J2: Conn_01x14, Connector_PinSocket_2.54mm:PinSocket_1x14_P2.54mm_Vertical_SMD_Pin1Left, symbol Connector_Generic:Conn_01x14
- added J3: OUT_1, MH_connectors:SAMESKY_TBLH10-508-02BK, symbol *partsbox:TBLH10-508-02BK
- added J4: OUT_2, MH_connectors:SAMESKY_TBLH10-508-02BK, symbol *partsbox:TBLH10-508-02BK
- added K1, K2: Relay_SPST_Latching_2coil, MH_switches:RELAY_G6CK-1117P-US_OMR, symbol *partsbox:G6CK-1117P-US-DC3
- added Q3, Q4: BC817, Package_TO_SOT_SMD:SOT-23, symbol *partsbox:BC817-40
- added R17: 0R, Resistor_SMD:R_0603_1608Metric, symbol *partsbox:0603-0ohm
- added R18, R19: 120R, Resistor_SMD:R_0603_1608Metric, symbol *partsbox:0603-120ohm
- added R8, R9: 4.7k, Resistor_SMD:R_0603_1608Metric, symbol *partsbox:0603-4.7Kohm
- added U11, U7: EL817, Package_DIP:SMDIP-4_W7.62mm, symbol *partsbox:EL8171S1(TU)-G
Connections:
- net +3V3: now also D1.1 (K), D2.1 (K), J1.2 (Pin_2), K1.A1, K1.B1, K2.A1, K2.B1, R17.2, R8.1, R9.1, U11.4, U7.4; no longer D5.2 (A)
- net ADDR_LED: now also J1.10 (Pin_10)
- net BTN1: now also J1.3 (Pin_3)
- net BTN2: now also J1.4 (Pin_4)
- net BTN3: now also J1.5 (Pin_5)
- net BTN4: now also J1.6 (Pin_6)
- net DISP_BUSY: now also J2.1 (Pin_1)
- net DISP_CS: now also J2.4 (Pin_4)
- net DISP_D/C: now also J2.3 (Pin_3)
- net DISP_RES: now also J2.2 (Pin_2)
- net DISP_SCLK: now also J2.5 (Pin_5)
- net DISP_SDA: now also J2.6 (Pin_6)
- net GND: now also J5.SH (Shield), BT5.2 (-), J1.11 (Pin_11), J1.14 (Pin_14), J2.12 (Pin_12), J2.14 (Pin_14), Q3.2 (E), Q4.2 (E), U11.2, U7.2
- net I2C_SCL: now also R9.2
- net I2C_SDA: now also R8.2
- net LED_G: now also J1.9 (Pin_9)
- net LED_PWM: now also J2.13 (Pin_13)
- net ONEWIRE: now also J2.7 (Pin_7)
- net PRESENCE_RX: now also J2.11 (Pin_11)
- net PRESENCE_TX: now also J2.10 (Pin_10)
- net SCL: now also J1.8 (Pin_8)
- net SDA: now also J1.7 (Pin_7)
- net TS_INT: now also J2.8 (Pin_8)
- net TS_RST: now also J2.9 (Pin_9)
- net VPP: now also J1.1 (Pin_1)
- net at D3.2 (A), Q2.3 (C): now also K2.B2
- net at D4.2 (A), Q1.3 (C): now also K2.A2
- net at D6.2 (A): now also BT5.1 (+)
- net PGOOD: now reaches U1.7 (~{PGOOD})
- net PGOOD: now also J1.12 (Pin_12)
- net CHG: now reaches U1.9 (~{CHG})
- net CHG: now also J1.13 (Pin_13)
- net RELAY2_RESET: now reaches U10.16 (IO46)
- net RELAY2_RESET: now also R19.1
- net RELAY2_SET: now reaches U10.26 (IO45)
- net RELAY2_SET: now also R18.1
- net RELAY_RESET renamed RELAY1_RESET
- net RELAY_SET renamed RELAY1_SET
- new net: D5.2 (A), R17.1
- new net: F2.1, J4.1 (Pin_1)
- new net: F2.2, K1.13
- new net: F1.1, J3.1 (Pin_1)
- new net: J3.2 (Pin_2), K2.14
- new net: R18.2, U7.1
- new net: Q3.1 (B), U7.3
- new net: Q4.1 (B), U11.3
- new net: D1.2 (A), K1.B2, Q4.3 (C)
- new net: R19.2, U11.1
- new net: D2.2 (A), K1.A2, Q3.3 (C)
- new net: J4.2 (Pin_2), K1.14
- new net: F1.2, K2.13
Other:
- note added: "Relays"
- note removed: "Relay"
- moved on the sheet: D3, D4, D5, Q1, Q2, R10, R11, TP8, U4, U5

Commit message: Push progress
Parts:
- removed J1, J2: Conn_01x14, Connector_PinSocket_2.54mm:PinSocket_1x14_P2.54mm_Vertical_SMD_Pin1Left, symbol Connector_Generic:Conn_01x14
- added J1: Conn_02x14_Top_Bottom, Connector_PinHeader_2.54mm:PinHeader_2x14_P2.54mm_Vertical_SMD, symbol Connector_Generic:Conn_02x14_Top_Bottom
Connections:
- net +3V3: now also J1.2 (Pin_2)
- net ADDR_LED: now also J1.10 (Pin_10)
- net BTN1: now also J1.3 (Pin_3)
- net BTN2: now also J1.4 (Pin_4)
- net BTN3: now also J1.5 (Pin_5)
- net BTN4: now also J1.6 (Pin_6)
- net CHG: now also J1.13 (Pin_13)
- net DISP_BUSY: now also J1.15 (Pin_15)
- net DISP_CS: now also J1.18 (Pin_18)
- net DISP_D/C: now also J1.17 (Pin_17)
- net DISP_RES: now also J1.16 (Pin_16)
- net DISP_SCLK: now also J1.19 (Pin_19)
- net DISP_SDA: now also J1.20 (Pin_20)
- net GND: now also J1.11 (Pin_11), J1.14 (Pin_14), J1.26 (Pin_26), J1.28 (Pin_28)
- net LED_G: now also J1.9 (Pin_9)
- net LED_PWM: now also J1.27 (Pin_27)
- net ONEWIRE: now also J1.21 (Pin_21)
- net PGOOD: now also J1.12 (Pin_12)
- net PRESENCE_RX: now also J1.25 (Pin_25)
- net PRESENCE_TX: now also J1.24 (Pin_24)
- net SCL: now also J1.8 (Pin_8)
- net SDA: now also J1.7 (Pin_7)
- net TS_INT: now also J1.22 (Pin_22)
- net TS_RST: now also J1.23 (Pin_23)
- net VPP: now also J1.1 (Pin_1)

Commit message: Start layout
Parts:
- removed F1, F2: 10A, Fuse:Fuse_Schurter_UMT250, symbol *partsbox:3403.0176.11
- removed J3: OUT_1, MH_connectors:SAMESKY_TBLH10-508-02BK, symbol *partsbox:TBLH10-508-02BK
- removed J4: OUT_2, MH_connectors:SAMESKY_TBLH10-508-02BK, symbol *partsbox:TBLH10-508-02BK
- added F1, F2: 10A, Fuse:Fuseholder_Clip-5x20mm_Littelfuse_111_Lateral_P18.80x5.00mm_D1.17mm_Horizontal, symbol *partsbox:01110501Z
- added J2: OUT_1, MH_connectors:CONN2_2604-1102_WAG, symbol *partsbox:2604-1102
- added J3: OUT_2, MH_connectors:CONN2_2604-1102_WAG, symbol *partsbox:2604-1102
Connections:
- net at K1.13: now also F2.2
- net at K2.14: now also J2.1 (Pin_1)
- net at K1.14: now also J3.1 (Pin_1)
- net at K2.13: now also F1.2
- new net: F1.1, J2.2 (Pin_2)
- new net: F2.1, J3.2 (Pin_2)

Commit message: Routing progress
Parts:
- removed U11, U4, U5, U7: EL817, Package_DIP:SMDIP-4_W7.62mm, symbol *partsbox:EL8171S1(TU)-G
- added U11, U4, U5, U7: LTV-217, Package_SO:SOP-4_4.4x2.6mm_P1.27mm, symbol *partsbox:LTV-217-B-G
- H1, H2, H3, H4: footprint MountingHole:MountingHole_3.2mm_M3_ISO7380_Pad_TopBottom -> MountingHole:MountingHole_3.2mm_M3_ISO7380
- J1: symbol Connector_Generic:Conn_02x14_Top_Bottom -> Connector_Generic:Conn_02x14_Odd_Even
Connections:
- net +3V3: now also J1.3 (Pin_3), U11.4, U4.4, U5.4, U7.4; no longer J1.2 (Pin_2)
- net ADDR_LED: now also J1.21 (Pin_21); no longer J1.10 (Pin_10)
- net BTN1: now also J1.9 (Pin_9), U10.35 (MTMS/IO42); no longer J1.3 (Pin_3), U10.34 (MTDI/IO41)
- net BTN2: now also J1.11 (Pin_11), U10.34 (MTDI/IO41); no longer J1.4 (Pin_4), U10.35 (MTMS/IO42)
- net BTN3: now also J1.13 (Pin_13), U10.33 (MTDO/IO40); no longer J1.5 (Pin_5), U10.24 (IO47)
- net BTN4: now also J1.15 (Pin_15), U10.32 (MTCK/IO39); no longer J1.6 (Pin_6), U10.25 (IO48)
- net CHG: now also J1.26 (Pin_26); no longer J1.13 (Pin_13)
- net DISP_BUSY: now also J1.2 (Pin_2); no longer J1.15 (Pin_15)
- net DISP_CS: now also J1.8 (Pin_8); no longer J1.18 (Pin_18)
- net DISP_D/C: now also J1.6 (Pin_6); no longer J1.17 (Pin_17)
- net DISP_RES: now also J1.4 (Pin_4); no longer J1.16 (Pin_16)
- net DISP_SCLK: now also J1.10 (Pin_10); no longer J1.19 (Pin_19)
- net DISP_SDA: now also J1.12 (Pin_12); no longer J1.20 (Pin_20)
- net GND: now also J1.22 (Pin_22), J1.23 (Pin_23), J1.27 (Pin_27), U11.2, U4.2, U5.2, U7.2; no longer J1.11 (Pin_11), J1.14 (Pin_14), J1.26 (Pin_26)
- net I2C_SCL: now also J1.7 (Pin_7)
- net I2C_SDA: now also J1.5 (Pin_5)
- net LED_G: no longer J1.9 (Pin_9), U10.32 (MTCK/IO39)
- net LED_PWM: now also J1.25 (Pin_25); no longer J1.27 (Pin_27), U10.33 (MTDO/IO40)
- net ONEWIRE: now also J1.14 (Pin_14); no longer J1.21 (Pin_21)
- net PGOOD: now also J1.24 (Pin_24); no longer J1.12 (Pin_12)
- net PRESENCE_RX: now also J1.17 (Pin_17); no longer J1.25 (Pin_25)
- net PRESENCE_TX: now also J1.19 (Pin_19); no longer J1.24 (Pin_24)
- net RELAY1_RESET: now also U10.24 (IO47); no longer U10.6 (IO6)
- net RELAY1_SET: now also U10.23 (IO21); no longer U10.5 (IO5)
- net RELAY2_RESET: now also U10.25 (IO48); no longer U10.16 (IO46)
- net RTC_INT: now also U10.5 (IO5); no longer U10.23 (IO21)
- net TS_INT: now also J1.16 (Pin_16); no longer J1.22 (Pin_22)
- net TS_RST: now also J1.18 (Pin_18); no longer J1.23 (Pin_23)
- net at R10.2: now also U4.1
- net at Q1.1 (B): now also U4.3
- net at R11.2: now also U5.1
- net at R18.2: now also U7.1
- net at Q3.1 (B): now also U7.3
- net at Q4.1 (B): now also U11.3
- net at R19.2: now also U11.1
- net at Q2.1 (B): now also U5.3
- net SCL: no longer names the net of U10.22 (IO14)
- net SCL: no longer J1.8 (Pin_8)
- net SDA: no longer names the net of U10.8 (IO15)
- net SDA: no longer J1.7 (Pin_7)
