File: V2/main_board/main_board.kicad_sch (KiCad schematic)
At the start: 102 parts, among them J1 USB_C_Receptacle_USB2.0_16P, J2 OUT_1, J3 Conn_02x14_Top_Bottom, J4 OUT_2, J5 EXT_TEMP, K1 Relay_SPST_Latching_2coil, K2 Relay_SPST_Latching_2coil, Q1 2N7002, Q2 BC817, Q3 BC817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

Commit message: fix symbol
Parts:
- added C16: 100nF, Capacitor_SMD:C_0603_1608Metric, symbol *partsbox:0603-100nF
- added D10, D8, D9: D_TVS, Diode_SMD:D_SOD-323, symbol *partsbox:H8VHD3B
- added FB3: FerriteBead_Small, Inductor_SMD:L_0603_1608Metric, symbol *partsbox:BLM18PG121SN1D
Connections:
- net +3V3: now also D9.2 (A2)
- net GND: now also C16.2, D10.1 (A1), D8.1 (A1), D9.1 (A1), FB3.2; no longer J5.3 (Pin_3), J5.SH (Shield)
- net ONEWIRE: now also D8.2 (A2)
- new net: C16.1, D10.2 (A2), FB3.1, J5.3 (Pin_3), J5.SH (Shield)
Other:
- moved on the sheet: C14, C15, J5, U12, U13

Commit message: Fixes
Parts:
- removed TP2: IO3, TestPoint:TestPoint_Pad_2.0x2.0mm, symbol Connector:TestPoint
Connections:
- net GND: no longer J3.23 (Pin_23)
- net PRESENCE_OUT: now reaches U4.6 (IO6)
- net PRESENCE_OUT: now also J3.23 (Pin_23)
Changed lines of the file:
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@@
 	)
 	(junction
-		(at 369.57 66.04)
-		(diameter 0)
-		(color 0 0 0 0)
-	)
-	(junction
 		(at 241.3 31.75)
 		(diameter 0)
@@
 	(wire
 		(pts
-			(xy 359.41 63.5) (xy 372.11 63.5)
+			(xy 358.14 63.5) (xy 372.11 63.5)
 		)
 		(stroke
@@
 	(wire
 		(pts
-			(xy 359.41 40.64) (xy 372.11 40.64)
+			(xy 358.14 40.64) (xy 372.11 40.64)
 		)
 		(stroke
@@
 	(wire
 		(pts
-			(xy 359.41 50.8) (xy 372.11 50.8)
+			(xy 358.14 50.8) (xy 372.11 50.8)
 		)
 		(stroke
@@
 	(wire
 		(pts
-			(xy 369.57 60.96) (xy 369.57 66.04)
-		)
-		(stroke
-			(width 0)
-			(type default)
-		)
-	)
-	(wire
-		(pts
 			(xy 325.12 40.64) (xy 325.12 45.72)
 		)
@@
 	(wire
 		(pts
-			(xy 359.41 43.18) (xy 372.11 43.18)
+			(xy 358.14 43.18) (xy 372.11 43.18)
 		)
 		(stroke
@@
 	(wire
 		(pts
-			(xy 359.41 53.34) (xy 372.11 53.34)
+			(xy 358.14 53.34) (xy 372.11 53.34)
 		)
 		(stroke
@@
 	(wire
 		(pts
+			(xy 358.14 60.96) (xy 372.11 60.96)
+		)
+		(stroke
+			(width 0)
+			(type default)
+		)
+	)
+	(wire
+		(pts
 			(xy 124.46 234.95) (xy 149.86 234.95)
 		)
@@
 	(wire
 		(pts
-			(xy 359.41 48.26) (xy 372.11 48.26)
+			(xy 358.14 48.26) (xy 372.11 48.26)
 		)
 		(stroke
@@
 	(wire
 		(pts
+			(xy 132.08 181.61) (xy 149.86 181.61)
+		)
+		(stroke
+			(width 0)
+			(type default)
+		)
+	)
+	(wire
+		(pts
 			(xy 116.84 124.46) (xy 116.84 127)
 		)
@@
 	(wire
 		(pts
-			(xy 359.41 38.1) (xy 372.11 38.1)
+			(xy 358.14 38.1) (xy 372.11 38.1)
 		)
 		(stroke
@@
 	(wire
 		(pts
-			(xy 359.41 55.88) (xy 372.11 55.88)
+			(xy 358.14 55.88) (xy 372.11 55.88)
 		)
 		(stroke
@@
 	(wire
 		(pts
-			(xy 110.49 181.61) (xy 149.86 181.61)
-		)
-		(stroke
-			(width 0)
-			(type default)
-		)
-	)
-	(wire
-		(pts
 			(xy 77.47 114.3) (xy 77.47 111.76)
 		)
@@
 	(wire
 		(pts
-			(xy 359.41 45.72) (xy 372.11 45.72)
+			(xy 358.14 45.72) (xy 372.11 45.72)
 		)
 		(stroke
@@
 	(wire
 		(pts
-			(xy 372.11 58.42) (xy 359.41 58.42)
+			(xy 372.11 58.42) (xy 358.14 58.42)
 		)
 		(stroke
@@
 	(wire
 		(pts
-			(xy 372.11 60.96) (xy 369.57 60.96)
-		)
-		(stroke
-			(width 0)
-			(type default)
-		)
-	)
-	(wire
-		(pts
 			(xy 149.86 191.77) (xy 132.08 191.77)
 		)
@@
 		)
 	)
+	(label "PRESENCE_OUT"
+		(at 132.08 181.61 0)
+		(effects
+			(font
+				(size 1.27 1.27)
+			)
+			(justify left bottom)
+		)
+	)
 	(label "SYSOFF"
 		(at 212.09 63.5 0)
@@
 	)
 	(label "I2C_SCL"
-		(at 359.41 40.64 0)
+		(at 358.14 40.64 0)
 		(effects
 			(font
@@
 		)
 	)
+	(label "PRESENCE_OUT"
+		(at 358.14 60.96 0)
+		(effects
+			(font
+				(size 1.27 1.27)
+			)
+			(justify left bottom)
+		)
+	)
 	(label "TS_INT"
 		(at 132.08 209.55 0)
@@
 	)
 	(label "BTN4"
-		(at 359.41 50.8 0)
+		(at 358.14 50.8 0)
 		(effects
 			(font
@@
 	)
 	(label "PRESENCE_TX"
-		(at 359.41 55.88 0)
+		(at 358.14 55.88 0)
 		(effects
 			(font
@@
 	)
 	(label "BTN3"
-		(at 359.41 48.26 0)
+		(at 358.14 48.26 0)
 		(effects
 			(font
@@
 	)
 	(label "BTN2"
-		(at 359.41 45.72 0)
+		(at 358.14 45.72 0)
 		(effects
 			(font
@@
 	)
 	(label "PRESENCE_RX"
-		(at 359.41 53.34 0)
+		(at 358.14 53.34 0)
 		(effects
 			(font
@@
 	)
 	(label "I2C_SDA"
-		(at 359.41 38.1 0)
+		(at 358.14 38.1 0)
 		(effects
 			(font
@@
 	)
 	(label "LED_PWM"
-		(at 359.41 63.5 0)
+		(at 358.14 63.5 0)
 		(effects
 			(font
@@
 	)
 	(label "BTN1"
-		(at 359.41 43.18 0)
+		(at 358.14 43.18 0)
 		(effects
 			(font
@@
 	)
 	(label "ADDR_LED"
-		(at 359.41 58.42 0)
+		(at 358.14 58.42 0)
 		(effects
 			(font
@@
 					(unit 1)
 				)
-			)
-		)
-	)
-	(symbol
-		(lib_id "Connector:TestPoint")
-		(at 110.49 181.61 90)
-		(unit 1)
-		(exclude_from_sim no)
-		(in_bom yes)
-		(on_board yes)
-		(dnp no)
-		(fields_autoplaced yes)
-		(property "Reference" "TP2"
-			(at 107.188 176.53 90)
-			(effects
-				(font
-					(size 1.27 1.27)
-				)
-			)
-		)
-		(property "Value" "IO3"
-			(at 107.188 179.07 90)
-			(effects
-				(font
-					(size 1.27 1.27)
-				)
-			)
-		)
-		(property "Footprint" "TestPoint:TestPoint_Pad_2.0x2.0mm"
-			(at 110.49 176.53 0)
-			(effects
-				(font
-					(size 1.27 1.27)
-				)
-				(hide yes)
-			)
-		)
-		(property "Datasheet" "~"
-			(at 110.49 176.53 0)
-			(effects
-				(font
-					(size 1.27 1.27)
-				)
-				(hide yes)
-			)
-		)
-		(property "Description" "test point"
-			(at 110.49 181.61 0)
-			(effects
-				(font
-					(size 1.27 1.27)
-				)
-				(hide yes)
-			)
-		)
-		(pin "1"
-		)
-		(instances
-			(project "main_board"
-				(path "/2310583b-51dd-4992-a296-db500aa0a56d"
-					(reference "TP2")
-					(unit 1)
-				)

Commit message: Redo high voltage
Connections:
- net RELAY2_RESET: now also U4.26 (IO45); no longer U4.25 (IO48)
- net RELAY2_SET: now also U4.25 (IO48); no longer U4.26 (IO45)
- net at F2.1: now also J2.1 (Pin_1); no longer J2.2 (Pin_2)
- net at K1.14: now also J2.2 (Pin_2); no longer J2.1 (Pin_1)
- net at J4.1 (Pin_1): now also F3.1; no longer K2.14
- net at J4.2 (Pin_2): now also K2.14; no longer F3.1
Changed lines of the file:
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@@
 		)
 	)
+	(label "RELAY2_SET"
+		(at 132.08 247.65 0)
+		(effects
+			(font
+				(size 1.27 1.27)
+			)
+			(justify left bottom)
+		)
+	)
 	(label "I2C_SDA"
 		(at 275.59 212.09 180)
@@
 		)
 	)
+	(label "RELAY2_RESET"
+		(at 132.08 240.03 0)
+		(effects
+			(font
+				(size 1.27 1.27)
+			)
+			(justify left bottom)
+		)
+	)
 	(label "BTN2"
 		(at 358.14 45.72 0)
@@
 		)
 	)
-	(label "RELAY2_RESET"
-		(at 132.08 247.65 0)
-		(effects
-			(font
-				(size 1.27 1.27)
-			)
-			(justify left bottom)
-		)
-	)
 	(label "BTN1"
 		(at 358.14 43.18 0)
@@
 		)
 	)
-	(label "RELAY2_SET"
-		(at 132.08 240.03 0)
-		(effects
-			(font
-				(size 1.27 1.27)
-			)
-			(justify left bottom)
-		)
-	)
 	(label "DISP_CS"
 		(at 397.51 40.64 180)
@@
 	(symbol
 		(lib_id "*partsbox:2604-1102")
-		(at 279.4 110.49 0)
+		(at 279.4 113.03 0)
+		(mirror x)
 		(unit 1)
 		(exclude_from_sim no)
@@
 		(on_board yes)
 		(dnp no)
-		(fields_autoplaced yes)
 		(property "Reference" "J2"
-			(at 281.94 110.4899 0)
+			(at 281.94 113.0301 0)
 			(effects
 				(font
@@
 		)
 		(property "Value" "OUT_1"
-			(at 281.94 113.0299 0)
+			(at 281.94 110.4901 0)
 			(effects
 				(font
@@
 		)
 		(property "Footprint" "MH_connectors:CONN2_2604-1102_WAG"
-			(at 279.4 110.49 0)
+			(at 279.4 113.03 0)
 			(effects
 				(font
@@
 		)
 		(property "Datasheet" "HTTPS://PARTSBOX.COM/I1KWDMV52F4H6V9WGVQNDT9J97J"
-			(at 279.4 110.49 0)
+			(at 279.4 113.03 0)
 			(effects
 				(font
@@
 		)
 		(property "Description" ""
-			(at 279.4 110.49 0)
+			(at 279.4 113.03 0)
 			(effects
 				(font
@@
 		)
 		(property "Type" "Linked"
-			(at 279.4 110.49 0)
+			(at 279.4 113.03 0)
 			(effects
 				(font
@@
 		)
 		(property "Manufacturer" "WAGO"
-			(at 279.4 110.49 0)
+			(at 279.4 113.03 0)
 			(effects
 				(font
@@
 		)
 		(property "MPN" "2604-1102"
-			(at 279.4 110.49 0)
+			(at 279.4 113.03 0)
 			(effects
 				(font
@@
 		)
 		(property "PartsBox ID" "1kwdmv52f4h6v9wgvqndt9j97j"
-			(at 279.4 110.49 0)
+			(at 279.4 113.03 0)
 			(effects
 				(font
@@
 		)
 		(instances
-			(project ""
+			(project "main_board"
 				(path "/2310583b-51dd-4992-a296-db500aa0a56d"
 					(reference "J2")
@@
 	(symbol
 		(lib_id "*partsbox:2604-1102")
-		(at 379.73 110.49 0)
+		(at 379.73 113.03 0)
+		(mirror x)
 		(unit 1)
 		(exclude_from_sim no)
@@
 		(on_board yes)
 		(dnp no)
-		(fields_autoplaced yes)
 		(property "Reference" "J4"
-			(at 382.27 110.4899 0)
+			(at 382.27 113.0301 0)
 			(effects
 				(font
@@
 		)
 		(property "Value" "OUT_2"
-			(at 382.27 113.0299 0)
+			(at 382.27 110.4901 0)
 			(effects
 				(font
@@
 		)
 		(property "Footprint" "MH_connectors:CONN2_2604-1102_WAG"
-			(at 379.73 110.49 0)
+			(at 379.73 113.03 0)
 			(effects
 				(font
@@
 		)
 		(property "Datasheet" "HTTPS://PARTSBOX.COM/I1KWDMV52F4H6V9WGVQNDT9J97J"
-			(at 379.73 110.49 0)
+			(at 379.73 113.03 0)
 			(effects
 				(font
@@
 		)
 		(property "Description" ""
-			(at 379.73 110.49 0)
+			(at 379.73 113.03 0)
 			(effects
 				(font
@@
 		)
 		(property "Type" "Linked"
-			(at 379.73 110.49 0)
+			(at 379.73 113.03 0)
 			(effects
 				(font
@@
 		)
 		(property "Manufacturer" "WAGO"
-			(at 379.73 110.49 0)
+			(at 379.73 113.03 0)
 			(effects
 				(font
@@
 		)
 		(property "MPN" "2604-1102"
-			(at 379.73 110.49 0)
+			(at 379.73 113.03 0)
 			(effects
 				(font
@@
 		)
 		(property "PartsBox ID" "1kwdmv52f4h6v9wgvqndt9j97j"
-			(at 379.73 110.49 0)
+			(at 379.73 113.03 0)
 			(effects
 				(font

Commit message: More fixes
Parts:
- removed C6: 1uF, Capacitor_SMD:C_0603_1608Metric, symbol *partsbox:0603-100nF
- added C6: 1uF, Capacitor_SMD:C_0603_1608Metric, symbol *partsbox:0603-1uF
Connections:
- net +3V3: now also C6.1
- net GND: now also C6.2
Changed lines of the file:
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@@
 	)
 	(symbol
-		(lib_id "*partsbox:0603-100nF")
-		(at 102.87 160.02 180)
-		(unit 1)
-		(exclude_from_sim no)
-		(in_bom yes)
-		(on_board yes)
-		(dnp no)
-		(fields_autoplaced yes)
-		(property "Reference" "C6"
-			(at 106.68 158.7499 0)
-			(effects
-				(font
-					(size 1.27 1.27)
-				)
-				(justify right)
-			)
-		)
-		(property "Value" "1uF"
-			(at 106.68 161.2899 0)
-			(effects
-				(font
-					(size 1.27 1.27)
-				)
-				(justify right)
-			)
-		)
-		(property "Footprint" "Capacitor_SMD:C_0603_1608Metric"
-			(at 101.9048 156.21 0)
-			(effects
-				(font
-					(size 1.27 1.27)
-				)
-				(hide yes)
-			)
-		)
-		(property "Datasheet" "HTTPS://PARTSBOX.COM/I6AFR1F2MY2JJJ8VS6V1P4RPR25"
-			(at 102.87 160.02 0)
-			(effects
-				(font
-					(size 1.27 1.27)
-				)
-				(hide yes)
-			)
-		)
-		(property "Description" ""
-			(at 102.87 160.02 0)
-			(effects
-				(font
-					(size 1.27 1.27)
-				)
-				(hide yes)
-			)
-		)
-		(property "Type" "Meta"
-			(at 102.87 160.02 0)
-			(effects
-				(font
-					(size 1.27 1.27)
-				)
-				(hide yes)
-			)
-		)
-		(property "Manufacturer" ""
-			(at 102.87 160.02 0)
-			(effects
-				(font
-					(size 1.27 1.27)
-				)
-				(hide yes)
-			)
-		)
-		(property "MPN" ""
-			(at 102.87 160.02 0)
-			(effects
-				(font
-					(size 1.27 1.27)
-				)
-				(hide yes)
-			)
-		)
-		(property "PartsBox ID" "6afr1f2my2jjj8vs6v1p4rpr25"
-			(at 102.87 160.02 0)
-			(effects
-				(font
-					(size 1.27 1.27)
-				)
-				(hide yes)
-			)
-		)
-		(pin "1"
-		)
-		(pin "2"
-		)
-		(instances
-			(project "main_board"
-				(path "/2310583b-51dd-4992-a296-db500aa0a56d"
-					(reference "C6")
-					(unit 1)
-				)
-			)
-		)
-	)
-	(symbol
 		(lib_id "power:GND")
 		(at 162.56 257.81 0)
@@
 					(unit 1)
 				)
+			)
+		)
+	)
+	(symbol
+		(lib_id "*partsbox:0603-1uF")
+		(at 102.87 160.02 0)
+		(unit 1)
+		(exclude_from_sim no)
+		(in_bom yes)
+		(on_board yes)
+		(dnp no)
+		(fields_autoplaced yes)
+		(property "Reference" "C6"
+			(at 106.68 158.7499 0)
+			(effects
+				(font
+					(size 1.27 1.27)
+				)
+				(justify left)
+			)
+		)
+		(property "Value" "1uF"
+			(at 106.68 161.2899 0)
+			(effects
+				(font
+					(size 1.27 1.27)
+				)
+				(justify left)
+			)
+		)
+		(property "Footprint" "Capacitor_SMD:C_0603_1608Metric"
+			(at 103.8352 163.83 0)
+			(effects
+				(font
+					(size 1.27 1.27)
+				)
+				(hide yes)
+			)
+		)
+		(property "Datasheet" "HTTPS://PARTSBOX.COM/I6KADBS4VVEKM59A2TDN2X98YMN"
+			(at 102.87 160.02 0)
+			(effects
+				(font
+					(size 1.27 1.27)
+				)
+				(hide yes)
+			)
+		)
+		(property "Description" ""
+			(at 102.87 160.02 0)
+			(effects
+				(font
+					(size 1.27 1.27)
+				)
+				(hide yes)
+			)
+		)
+		(property "Type" "Meta"
+			(at 102.87 160.02 0)
+			(effects
+				(font
+					(size 1.27 1.27)
+				)
+				(hide yes)
+			)
+		)
+		(property "Manufacturer" ""
+			(at 102.87 160.02 0)
+			(effects
+				(font
+					(size 1.27 1.27)
+				)
+				(hide yes)
+			)
+		)
+		(property "MPN" ""
+			(at 102.87 160.02 0)
+			(effects
+				(font
+					(size 1.27 1.27)
+				)
+				(hide yes)
+			)
+		)
+		(property "PartsBox ID" "6kadbs4vvekm59a2tdn2x98ymn"
+			(at 102.87 160.02 0)
+			(effects
+				(font
+					(size 1.27 1.27)
+				)
+				(hide yes)
+			)
+		)
+		(pin "2"
+		)
+		(pin "1"
+		)
+		(instances
+			(project "main_board"
+				(path "/2310583b-51dd-4992-a296-db500aa0a56d"
+					(reference "C6")
+					(unit 1)
+				)
