File: V2/main_board/main_board.kicad_pcb (KiCad board)
At the start: 2 copper layers, 100 x 103.5 mm, 104 parts, among them J1 USB_C_Receptacle_USB2.0_16P, J2 OUT_1, J3 Conn_02x14_Top_Bottom, J4 OUT_2, J5 EXT_TEMP, K1 Relay_SPST_Latching_2coil, K2 Relay_SPST_Latching_2coil, Q1 2N7002, Q2 BC817, Q3 BC817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

Commit message: Fixes
Parts:
- removed TP2: IO3, TestPoint:TestPoint_Pad_2.0x2.0mm
- added C16: 100nF, Capacitor_SMD:C_0603_1608Metric, F.Cu at (87.2, 74.2)
- added D10: D_TVS, Diode_SMD:D_SOD-323, F.Cu at (90.8, 75.0)
- added D8: D_TVS, Diode_SMD:D_SOD-323, F.Cu at (93.2, 75.0)
- added D9: D_TVS, Diode_SMD:D_SOD-323, F.Cu at (95.8, 75.0)
- added FB3: FerriteBead_Small, Inductor_SMD:L_0603_1608Metric, F.Cu at (88.8, 74.2)
- moved R16 1.00 mm to (90.0, 79.0)
- moved REF** 0.56 mm to (136.0, 54.0)
Connections:
- J3 pad 23: GND -> /PRESENCE_OUT
- J5 pad 3: GND -> Net-(D10-A2)
- J5 pad SH: GND -> Net-(D10-A2)
- U4 pad 6: Net-(U4-IO6) -> /PRESENCE_OUT
Routing:
- net /PRESENCE_OUT: track 0.00 -> 33.8 mm, vias 0 -> 2
- net /I2C_SCL: track 151.2 -> 134.9 mm
- net /I2C_SDA: track 160.7 -> 146.8 mm
- net VPP: track 115.0 -> 101.6 mm
- net /ONEWIRE: track 137.6 -> 125.9 mm, vias 8 -> 5
- net Net-(U4-IO6): track 9.54 -> 0.00 mm
- net GND: track 18.2 -> 26.1 mm, vias 118 -> 135
- net /DISP_D/C: track 50.6 -> 43.8 mm
- net /LED_PWM: track 15.9 -> 22.5 mm
- net /PRESENCE_TX: track 53.8 -> 59.1 mm
- net /PRESENCE_RX: track 55.7 -> 60.8 mm
- net /PGOOD: track 21.4 -> 26.5 mm
- net /CHG: track 20.2 -> 25.3 mm
- net /BTN3: track 51.2 -> 56.2 mm
- net /BTN1: track 61.5 -> 66.4 mm
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- added copper zone on F.Cu, net Net-(D10-A2)
Other:
- board text added: "2026"

Commit message: Final updates
Changed lines of the file:
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@@
 			(layer "F.Fab")
 		)
-		(fp_text user "*"
-			(at -10.16 -24.980001 270)
-			(layer "F.SilkS")
-			(effects
-				(font
-					(size 1 1)
-					(thickness 0.15)
-				)
-			)
-		)
-		(fp_text user "*"
-			(at -10.16 -24.980001 270)
-			(unlocked yes)
-			(layer "F.SilkS")
-			(effects
-				(font
-					(size 1 1)
-					(thickness 0.15)
-				)
-			)
-		)
 		(fp_text user "${REFERENCE}"
 			(at -5.08 -8.930001 0)
@@
 		)
 		(fp_text user "*"
-			(at -10.16 -24.980001 270)
-			(layer "F.SilkS")
-			(effects
-				(font
-					(size 1 1)
-					(thickness 0.15)
-				)
-			)
-		)
-		(fp_text user "*"
-			(at -10.16 -24.980001 270)
-			(unlocked yes)
-			(layer "F.SilkS")
-			(effects
-				(font
-					(size 1 1)
-					(thickness 0.15)
-				)
-			)
-		)
-		(fp_text user "*"
 			(at -10.16 -22.940001 270)
 			(layer "F.Fab")
@@
 		(at 111 134)
 		(property "Reference" "BT4"
-			(at 31.5 -8 0)
+			(at 31.5 -8 180)
 			(unlocked yes)
 			(layer "B.SilkS")
@@
 		(at 111 69.5)
 		(property "Reference" "BT1"
-			(at 31.5 -8 0)
+			(at 31.5 -8 180)
 			(unlocked yes)
 			(layer "B.SilkS")
@@
 		(at 111 91)
 		(property "Reference" "BT2"
-			(at 31.5 -8 0)
+			(at 31.5 -8 180)
 			(unlocked yes)
 			(layer "B.SilkS")
@@
 		(at 110.99 112.5)
 		(property "Reference" "BT3"
-			(at 34.26 -8 0)
+			(at 28.76 -8 180)
 			(unlocked yes)
 			(layer "B.SilkS")
