File: V2/main_board/main_board.kicad_pcb (KiCad board)
At the start: 2 copper layers, 100 x 103.5 mm, 108 parts, among them J1 USB_C_Receptacle_USB2.0_16P, J2 OUT_1, J3 Conn_02x14_Top_Bottom, J4 OUT_2, J5 EXT_TEMP, K1 Relay_SPST_Latching_2coil, K2 Relay_SPST_Latching_2coil, Q1 2N7002, Q2 BC817, Q3 BC817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

Commit message: Boards ordered
Other:
- board text removed: "JLCJLCJLCJLC"
Changed lines of the file:
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@@
 		(sheetname "/")
 		(sheetfile "main_board.kicad_sch")
-		(attr smd)
+		(attr smd exclude_from_pos_files exclude_from_bom)
 		(fp_line
 			(start 2.06 -2.56)
@@
 			(thermal_bridge_angle 45)
 		)
-		(pad "41" thru_hole circle
-			(at -2.86 -0.66 180)
-			(size 0.6 0.6)
-			(drill 0.2)
-			(property pad_prop_heatsink)
-			(layers "*.Cu" "*.Mask")
-			(remove_unused_layers no)
-			(net 1 "GND")
-			(pinfunction "GND")
-			(pintype "passive")
-			(zone_connect 2)
-		)
 		(pad "41" smd rect
 			(at -2.86 0.09 180)
@@
 			(thermal_bridge_angle 45)
 		)
-		(pad "41" thru_hole circle
-			(at -2.86 0.84 180)
-			(size 0.6 0.6)
-			(drill 0.2)
-			(property pad_prop_heatsink)
-			(layers "*.Cu" "*.Mask")
-			(remove_unused_layers no)
-			(net 1 "GND")
-			(pinfunction "GND")
-			(pintype "passive")
-			(zone_connect 2)
-		)
 		(pad "41" smd rect
 			(at -2.86 1.59 180)
@@
 			(thermal_bridge_angle 45)
 		)
-		(pad "41" thru_hole circle
-			(at -2.11 -1.41 180)
-			(size 0.6 0.6)
-			(drill 0.2)
-			(property pad_prop_heatsink)
-			(layers "*.Cu" "*.Mask")
-			(remove_unused_layers no)
-			(net 1 "GND")
-			(pinfunction "GND")
-			(pintype "passive")
-			(zone_connect 2)
-		)
-		(pad "41" thru_hole circle
-			(at -2.11 0.09 180)
-			(size 0.6 0.6)
-			(drill 0.2)
-			(property pad_prop_heatsink)
-			(layers "*.Cu" "*.Mask")
-			(remove_unused_layers no)
-			(net 1 "GND")
-			(pinfunction "GND")
-			(pintype "passive")
-			(zone_connect 2)
-		)
-		(pad "41" thru_hole circle
-			(at -2.11 1.59 180)
-			(size 0.6 0.6)
-			(drill 0.2)
-			(property pad_prop_heatsink)
-			(layers "*.Cu" "*.Mask")
-			(remove_unused_layers no)
-			(net 1 "GND")
-			(pinfunction "GND")
-			(pintype "passive")
-			(zone_connect 2)
-		)
 		(pad "41" smd rect
 			(at -1.36 -1.41 180)
@@
 			(thermal_bridge_angle 45)
 		)
-		(pad "41" thru_hole circle
-			(at -1.36 -0.66 180)
-			(size 0.6 0.6)
-			(drill 0.2)
-			(property pad_prop_heatsink)
-			(layers "*.Cu" "*.Mask")
-			(remove_unused_layers no)
-			(net 1 "GND")
-			(pinfunction "GND")
-			(pintype "passive")
-			(zone_connect 2)
-		)
 		(pad "41" smd rect
 			(at -1.36 0.09 180)
@@
 			(thermal_bridge_angle 45)
 		)
-		(pad "41" thru_hole circle
-			(at -1.36 0.84 180)
-			(size 0.6 0.6)
-			(drill 0.2)
-			(property pad_prop_heatsink)
-			(layers "*.Cu" "*.Mask")
-			(remove_unused_layers no)
-			(net 1 "GND")
-			(pinfunction "GND")
-			(pintype "passive")
-			(zone_connect 2)
-		)
 		(pad "41" smd rect
 			(at -1.36 1.59 180)
@@
 			(thermal_bridge_angle 45)
 		)
-		(pad "41" thru_hole circle
-			(at -0.61 -1.41 180)
-			(size 0.6 0.6)
-			(drill 0.2)
-			(property pad_prop_heatsink)
-			(layers "*.Cu" "*.Mask")
-			(remove_unused_layers no)
-			(net 1 "GND")
-			(pinfunction "GND")
-			(pintype "passive")
-			(zone_connect 2)
-		)
-		(pad "41" thru_hole circle
-			(at -0.61 0.09 180)
-			(size 0.6 0.6)
-			(drill 0.2)
-			(property pad_prop_heatsink)
-			(layers "*.Cu" "*.Mask")
-			(remove_unused_layers no)
-			(net 1 "GND")
-			(pinfunction "GND")
-			(pintype "passive")
-			(zone_connect 2)
-		)
-		(pad "41" thru_hole circle
-			(at -0.61 1.59 180)
-			(size 0.6 0.6)
-			(drill 0.2)
-			(property pad_prop_heatsink)
-			(layers "*.Cu" "*.Mask")
-			(remove_unused_layers no)
-			(net 1 "GND")
-			(pinfunction "GND")
-			(pintype "passive")
-			(zone_connect 2)
-		)
 		(pad "41" smd rect
 			(at 0.14 -1.41 180)
@@
 			(thermal_bridge_angle 45)
 		)
-		(pad "41" thru_hole circle
-			(at 0.14 -0.66 180)
-			(size 0.6 0.6)
-			(drill 0.2)
-			(property pad_prop_heatsink)
-			(layers "*.Cu" "*.Mask")
-			(remove_unused_layers no)
-			(net 1 "GND")
-			(pinfunction "GND")
-			(pintype "passive")
-			(zone_connect 2)
-		)
 		(pad "41" smd rect
 			(at 0.14 0.09 180)
@@
 			(thermal_bridge_angle 45)
 		)
-		(pad "41" thru_hole circle
-			(at 0.14 0.84 180)
-			(size 0.6 0.6)
-			(drill 0.2)
-			(property pad_prop_heatsink)
-			(layers "*.Cu" "*.Mask")
-			(remove_unused_layers no)
-			(net 1 "GND")
-			(pinfunction "GND")
-			(pintype "passive")
-			(zone_connect 2)
-		)
 		(pad "41" smd rect
 			(at 0.14 1.59 180)
@@
 			)
 		)
-		(property "LCSC" "C2927799"
+		(property "LCSC" ""
 			(at 0 0 0)
 			(layer "F.SilkS")
@@
 		(sheetname "/")
 		(sheetfile "main_board.kicad_sch")
-		(attr smd)
+		(attr smd exclude_from_pos_files exclude_from_bom)
 		(fp_line
 			(start -0.91 -1.56)
@@
 			)
 		)
-		(property "LCSC" "C2830320"
+		(property "LCSC" ""
 			(at 0 0 0)
 			(layer "F.SilkS")
@@
 		(sheetname "/")
 		(sheetfile "main_board.kicad_sch")
-		(attr smd)
+		(attr smd exclude_from_pos_files exclude_from_bom)
 		(fp_line
 			(start -0.91 -1.56)
@@
 		(sheetname "/")
 		(sheetfile "main_board.kicad_sch")
-		(attr smd)
+		(attr smd exclude_from_pos_files exclude_from_bom)
 		(fp_line
 			(start 2.06 2.56)
@@
 		)
 	)
-	(gr_text "JLCJLCJLCJLC"
-		(at 98.25 141 90)
-		(layer "F.SilkS")
-		(effects
-			(font
-				(size 2 2)
-				(thickness 0.2)
-			)
-		)
-	)
