File: V2/display_board/display_board.kicad_sch (KiCad schematic)
At the start: 64 parts, among them J5 Conn_02x14_Top_Bottom, Q1 Si1308EDL, SW1 SW_Push, SW2 SW_Push, SW3 SW_Push, SW4 SW_Push, U1 TPS61165DBV, U2 LTR-303ALS-01, U3 DS18B20Z, U4 SHT4x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

Commit message: Final updates
Parts:
- renumbered J5 to J1
Changed lines of the file:
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@@
 		(dnp no)
 		(fields_autoplaced yes)
-		(property "Reference" "J5"
+		(property "Reference" "J1"
 			(at 200.66 116.84 0)
 			(effects
@@
 			(project "display_board"
 				(path "/b4a04f60-fca9-4e45-9f9f-b48317aec4e2"
-					(reference "J5")
+					(reference "J1")
 					(unit 1)
 				)

Commit message: Update connectors
Parts:
- FL1, TS1: footprint Connector_FFC-FPC:Hirose_FH12-6S-0.5SH_1x06-1MP_P0.50mm_Horizontal -> MH_connectors:AFC24-S06FIA-00
- P1: footprint Connector_FFC-FPC:Hirose_FH12-24S-0.5SH_1x24-1MP_P0.50mm_Horizontal -> MH_connectors:AFC24-S24FIA-00
Changed lines of the file:
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@@
 			)
 		)
-		(property "Footprint" "Connector_FFC-FPC:Hirose_FH12-24S-0.5SH_1x24-1MP_P0.50mm_Horizontal"
+		(property "Footprint" "MH_connectors:AFC24-S24FIA-00"
 			(at 116.84 58.42 0)
 			(effects
@@
 			)
 		)
-		(property "Footprint" "Connector_FFC-FPC:Hirose_FH12-6S-0.5SH_1x06-1MP_P0.50mm_Horizontal"
+		(property "Footprint" "MH_connectors:AFC24-S06FIA-00"
 			(at 50.8 184.15 0)
 			(effects
@@
 			)
 		)
-		(property "Footprint" "Connector_FFC-FPC:Hirose_FH12-6S-0.5SH_1x06-1MP_P0.50mm_Horizontal"
+		(property "Footprint" "MH_connectors:AFC24-S06FIA-00"
 			(at 111.76 132.08 0)
 			(effects
