File: V2/display_board/display_board.kicad_pcb (KiCad board)
At the start: 2 copper layers, 100 x 103.5 mm, 66 parts, among them J1 Conn_02x14_Top_Bottom, Q1 Si1308EDL, SW1 SW_Push, SW2 SW_Push, SW3 SW_Push, SW4 SW_Push, U1 TPS61165DBV, U2 LTR-303ALS-01, U3 DS18B20Z, U4 SHT4x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

Commit message: Boards ordered
Other:
- board text removed: "JLCJLCJLCJLC"
Changed lines of the file:
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@@
 			)
 		)
+		(property "LCSC" ""
+			(at 0 0 0)
+			(layer "B.SilkS")
+			(hide yes)
+			(effects
+				(font
+					(size 1.27 1.27)
+					(thickness 0.15)
+				)
+			)
+		)
 		(property ki_fp_filters "Diode_SMD:D_SOD-123")
 		(sheetname "/")
 		(sheetfile "display_board.kicad_sch")
-		(attr smd)
+		(attr smd exclude_from_pos_files exclude_from_bom)
 		(fp_line
 			(start -2.36 -1)
@@
 		(sheetname "/")
 		(sheetfile "display_board.kicad_sch")
-		(attr smd)
+		(attr smd exclude_from_pos_files exclude_from_bom)
 		(fp_line
 			(start -0.91 1.56)
@@
 		(sheetname "/")
 		(sheetfile "display_board.kicad_sch")
-		(attr smd)
+		(attr smd exclude_from_pos_files exclude_from_bom)
 		(fp_line
 			(start -2.06 -2.56)
@@
 			)
 		)
-		(property "LCSC" "C77336"
+		(property "LCSC" ""
 			(at 0 0 0)
 			(layer "B.SilkS")
@@
 		(sheetname "/")
 		(sheetfile "display_board.kicad_sch")
-		(attr smd)
+		(attr smd exclude_from_pos_files exclude_from_bom)
 		(fp_line
 			(start -2.36 -1)
@@
 			)
 		)
+		(property "LCSC" ""
+			(at 0 0 0)
+			(layer "B.SilkS")
+			(hide yes)
+			(effects
+				(font
+					(size 1.27 1.27)
+					(thickness 0.15)
+				)
+			)
+		)
 		(property ki_fp_filters "Diode_SMD:D_SOD-123")
 		(sheetname "/")
 		(sheetfile "display_board.kicad_sch")
-		(attr smd)
+		(attr smd exclude_from_pos_files exclude_from_bom)
 		(fp_line
 			(start -2.36 1)
@@
 			)
 			(justify bottom)
-		)
-	)
-	(gr_text "JLCJLCJLCJLC"
-		(at 100 71.25 0)
-		(layer "F.SilkS")
-		(effects
-			(font
-				(size 1.25 1.25)
-				(thickness 0.125)
-			)
-			(justify bottom)

Commit message: Update connectors
Parts:
- FL1, TS1: footprint Connector_FFC-FPC:Hirose_FH12-6S-0.5SH_1x06-1MP_P0.50mm_Horizontal -> MH_connectors:AFC24-S06FIA-00
- P1: footprint Connector_FFC-FPC:Hirose_FH12-24S-0.5SH_1x24-1MP_P0.50mm_Horizontal -> MH_connectors:AFC24-S24FIA-00
- moved FL1 1.95 mm to (90.5, 110.2)
- moved P1 1.85 mm to (78.8, 124.8)
- moved TS1 1.85 mm to (134.0, 95.3)

Commit message: Update footprint
Parts:
- moved P1 1.58 mm to (78.8, 126.4), turned to 0 degrees
- moved TS1 1.57 mm to (134.0, 96.9), turned to 0 degrees
- moved FL1 1.52 mm to (90.5, 111.8), turned to 0 degrees
Connections:
- FL1 pad MP: GND -> (no net)
- P1 pad MP: GND -> (no net)
- TS1 pad MP: GND -> (no net)
